Commit message: Changed position of Camera from hand_tcp to hand (close to link_8) and changed the mount 180 degrees

File: src/franka_description/robots/common/franka_hand.xacro (robot description, xacro)
@@ -10,9 +10,4 @@
       </joint>
     </xacro:unless>
-    <xacro:property name="PI" value="3.1415926535897931"/>
-    <xacro:include filename="$(find franka_description)/robots/common/_d435.urdf.xacro" />
-    <xacro:sensor_d435 parent="${arm_id}_hand_tcp">
-          <origin xyz="-0.015 0 0.025" rpy="${PI} ${-PI/2} 0" /> <!-- <origin xyz="0.05 0 -0.14" rpy="${PI} ${-PI/2} 0" /> -->
-    </xacro:sensor_d435>
     <xacro:link_with_sc name="hand" gazebo="${gazebo}">
       <self_collision_geometries>

File: src/franka_description/robots/common/franka_robot.xacro (robot description, xacro)
@@ -14,4 +14,10 @@
     <xacro:include filename="$(find franka_description)/robots/common/franka_arm.xacro" />
     <xacro:franka_arm arm_id="${arm_id}" safety_distance="0.03" gazebo="$(arg gazebo)" joint_limits="${joint_limits}"/>
+    <!-- ADD REALSENSE D435 SENSOR HERE!!! -->
+    <xacro:property name="PI" value="3.1415926535897931"/>
+    <xacro:include filename="$(find franka_description)/robots/common/_d435.urdf.xacro" />
+    <xacro:sensor_d435 parent="${arm_id}_hand"><!-- <xacro:sensor_d435 parent="${arm_id}_hand_tcp"> -->
+          <origin xyz="0.10 0.0 0.0" rpy="0 ${-PI/2} 0" /> <!--  <origin xyz="-0.015 0 0.025" rpy="${PI} ${-PI/2} 0" />  <origin xyz="0.05 0 -0.14" rpy="${PI} ${-PI/2} 0" /> -->
+    </xacro:sensor_d435>
     <xacro:if value="$(arg hand)">
       <xacro:include filename="$(find franka_description)/robots/common/franka_hand.xacro"/>
