Commit message: Updated coordinate frame generation code, Now uses KDL to calculate new frames
Using KDL to create frames and multiply to get correct final frame poses to be sent to the robot.

File: src/franka_description/robots/common/franka_robot.xacro (robot description, xacro)
@@ -18,5 +18,5 @@
     <xacro:include filename="$(find franka_description)/robots/common/_d435.urdf.xacro" />
     <xacro:sensor_d435 parent="${arm_id}_hand"><!-- <xacro:sensor_d435 parent="${arm_id}_hand_tcp"> -->
-          <origin xyz="0.10 0.0 0.0" rpy="0 ${-PI/2} 0" /> <!--  <origin xyz="-0.015 0 0.025" rpy="${PI} ${-PI/2} 0" />  <origin xyz="0.05 0 -0.14" rpy="${PI} ${-PI/2} 0" /> -->
+      <origin xyz="0.1 0.0 0.0" rpy="0 ${-PI/2} 0" /> <!-- coordinates wrt parent link  <origin xyz="-0.015 0 0.025" rpy="${PI} ${-PI/2} 0" />  <origin xyz="0.05 0 -0.14" rpy="${PI} ${-PI/2} 0" /> -->
     </xacro:sensor_d435>
     <xacro:if value="$(arg hand)">

Commit message: Bugfix: Fixed camera's orientation

File: src/franka_description/robots/common/franka_robot.xacro (robot description, xacro)
@@ -18,5 +18,5 @@
     <xacro:include filename="$(find franka_description)/robots/common/_d435.urdf.xacro" />
     <xacro:sensor_d435 parent="${arm_id}_hand"><!-- <xacro:sensor_d435 parent="${arm_id}_hand_tcp"> -->
-      <origin xyz="0.1 0.0 0.0" rpy="0 ${-PI/2} 0" /> <!-- coordinates wrt parent link  <origin xyz="-0.015 0 0.025" rpy="${PI} ${-PI/2} 0" />  <origin xyz="0.05 0 -0.14" rpy="${PI} ${-PI/2} 0" /> -->
+      <origin xyz="0.1 0.0 0.0" rpy="${PI} ${-PI/2} 0" /> <!-- coordinates wrt parent link  <origin xyz="-0.015 0 0.025" rpy="${PI} ${-PI/2} 0" />  <origin xyz="0.05 0 -0.14" rpy="${PI} ${-PI/2} 0" /> -->
     </xacro:sensor_d435>
     <xacro:if value="$(arg hand)">

Commit message: Adjusted position of camera based on the real Franka robot

File: src/franka_description/robots/common/franka_robot.xacro (robot description, xacro)
@@ -18,5 +18,5 @@
     <xacro:include filename="$(find franka_description)/robots/common/_d435.urdf.xacro" />
     <xacro:sensor_d435 parent="${arm_id}_hand"><!-- <xacro:sensor_d435 parent="${arm_id}_hand_tcp"> -->
-      <origin xyz="0.1 0.0 0.0" rpy="${PI} ${-PI/2} 0" /> <!-- coordinates wrt parent link  <origin xyz="-0.015 0 0.025" rpy="${PI} ${-PI/2} 0" />  <origin xyz="0.05 0 -0.14" rpy="${PI} ${-PI/2} 0" /> -->
+      <origin xyz="0.045 0.0 -0.035" rpy="${PI} ${-PI/2} 0" /> <!-- coordinates wrt parent link  <origin xyz="-0.015 0 0.025" rpy="${PI} ${-PI/2} 0" />  <origin xyz="0.05 0 -0.14" rpy="${PI} ${-PI/2} 0" /> -->
     </xacro:sensor_d435>
     <xacro:if value="$(arg hand)">
